Commit message: second

File: src/litearm_a10_description/urdf/LiteArm_A10_251224.urdf (robot description, URDF)
Before this commit: robot LiteArm_A10_251224, 16 links, 15 joints
Links:
- link r_joint5_link: mass 0.54640883 -> 0.50640883
Joints:
- joint r_joint1_joint: axis 0 1 0 -> 0 -1 0; limit lower=-3.0543 upper=1.6581 effort=75 velocity=6.0737 -> lower=-1.6581 upper=3.0543 effort=75 velocity=6.0737
- joint r_joint2_joint: axis 1 0 0 -> -1 0 0; limit lower=-2.8623 upper=0.27925 effort=75 velocity=6.0737 -> lower=-0.27925 upper=2.8623 effort=75 velocity=6.0737
- joint r_joint4_joint: axis 0 1 0 -> 0 -1 0; limit lower=-2.44 upper=1.57 effort=50 velocity=6.0737 -> lower=-1.57 upper=2.44 effort=50 velocity=6.0737
- joint r_joint5_joint: axis 0 0 1 -> 0 0 -1
- joint r_joint6_joint: axis 1 0 0 -> -1 0 0
- joint r_joint7_joint: axis 0 1 0 -> 0 -1 0
