Commit message: 2

File: src/litearm_a10_251125/urdf/LiteArm_A10_251125.urdf (robot description, URDF)
Before this commit: robot LiteArm_A10_251125, 24 links, 23 joints
Joints:
- joint l_joint2_joint: axis 1 0 0 -> -1 0 0; limit lower=-0.27925 upper=2.8623 effort=75 velocity=6.0737 -> lower=-2.8623 upper=0.27925 effort=75 velocity=6.0737
- joint l_joint3_joint: axis 0 0 1 -> 0 0 -1
- joint l_joint5_joint: axis 0 0 1 -> 0 0 -1
- joint l_joint6_joint: axis 1 0 0 -> -1 0 0
- joint r_joint2_joint: limit lower=-0.27925 upper=2.8623 effort=75 velocity=6.0737 -> lower=-2.8623 upper=0.27925 effort=75 velocity=6.0737
